Commit message: Add interactive UI panels, visual overlays, mesh-box collision, and Panda grasp demo
- viz/ui_panels.py: UIPanel with parameter sliders, play/pause, joint control
- viz/overlays.py: ContactForceOverlay (arrows), JointAxisOverlay, CollisionAABBOverlay
- contact/sdf.py: mesh_box vertex-vs-OBB narrow phase, improved box-box edge threshold
- contact/detection.py: mesh-box / box-mesh pair dispatch in ContactDetector
- contact/solver.py: two-pass effective mass, cross-robot filters, compute_all_rbd_contact_forces,
  fixed link velocity propagation for mimic/fixed joints
- examples/grasp_demo.py: Panda 7-DOF parallel-jaw gripper grasping a box with UI controls
- examples/interactive_demo.py: 3-mode interactive demo (pendulum, drop, arm) with live parameter tuning
- Panda URDF: added per-link inertial properties for physically accurate dynamics

Co-Authored-By: Claude Opus 4.6 <noreply@anthropic.com>

File: examples/urdf/panda/panda.urdf (robot description, URDF)
Before this commit: robot panda, 12 links, 11 joints
Links:
- link panda_hand: mass None -> 0.73
- link panda_leftfinger: mass None -> 0.015
- link panda_link0: mass None -> 0.629769
- link panda_link1: mass None -> 4.970684
- link panda_link2: mass None -> 0.646926
- link panda_link3: mass None -> 3.228604
- link panda_link4: mass None -> 3.587895
- link panda_link5: mass None -> 1.225946
- link panda_link6: mass None -> 1.666555
- link panda_link7: mass None -> 0.735522
- link panda_rightfinger: mass None -> 0.015
