Commit message: feat: Scene API, RL infra, contact solver overhaul, mpm-grasp grip fix
Snapshot of the mpm-publish line of work. Grouped themes:

- Scene API (scene/{scene,runner}.py): declarative builder for
  robot/body/contact/grip; runner owns substep loop + kinematic grip
  with PD-target floor (replaces hand-rolled grasp loops). Examples
  reduced to ~40 lines of user code.

- examples/: relocate every demo into examples/pure_simulation/;
  delete the legacy 791-line grasp_demo.py (superseded by 134-line
  grasp_scene.py). Header docstrings + paper/README cross-refs
  updated.

- examples/pure_simulation/mpm_grasp_drop.py: align finger PD
  (kp 5e4->800), CLOSE/LIFT/MOVE finger q (+/-0.020 -> +/-0.011),
  add grip-time PD lock as a *floor* (max(traj, lock)) so the post-
  release inward spike disappears and the trajectory hands off
  smoothly when it rises above the snapshot.

- envs/ + examples/rl/: Gymnasium wrapper + SB3 PPO train/eval
  scripts, monitor logging.

- physics/contact/: constraint-based Coulomb-cone solver alongside
  penalty (constraint_solver.py + test_constraint_friction.py),
  link-frame contact + SLAB_PAD, AABB-aware narrowphase pruning,
  inlined SDF fast paths.

- physics/mpm/: Taichi MLS-MPM port (taichi_solver.py +
  test_mpm_taichi.py), vectorised P2G/G2P 27-stencil loops, AABB
  early-exit in collider, shrunk grasp-drop domain.

- physics/rbd, math/, model/robot.py: cached spatial transforms,
  Transform._fast() bypassing __post_init__, manual cross3, FK and
  joint-spatial-transform caches keyed on q-snapshot equality.

- paper/: ICRA positioning, gap analysis, CB novelty, references.

- 228 tests pass + 7 skipped.

Co-Authored-By: Claude Opus 4.7 <noreply@anthropic.com>

File: examples/pure_simulation/urdf/arm6_gripper/arm6_gripper.urdf (robot description, URDF)
Before this commit: robot arm6_gripper, 8 links, 7 joints
Links:
- link left_finger: geometry collision box size=0.080 0.010 0.040; visual box size=0.080 0.010 0.040
- link right_finger: geometry collision box size=0.080 0.010 0.040; visual box size=0.080 0.010 0.040

Commit message: Add deformable CB gripper contact and split grasp_scene physics flags.
Mount fingers at the palm tip, shift the grasp target, and wire
--object/--finger so rigid objects can be grasped with cantilever-bending
CB fingers via contact_deformable_gripper.

Co-authored-by: Cursor <cursoragent@cursor.com>

File: examples/pure_simulation/urdf/arm6_gripper/arm6_gripper.urdf (robot description, URDF)
Before this commit: robot arm6_gripper, 8 links, 7 joints
Joints:
- joint joint_left: origin xyz=0 0.043 0 rpy=0 0 0 -> xyz=0.025 0.043 0 rpy=0 0 0
- joint joint_right: origin xyz=0 -0.043 0 rpy=0 0 0 -> xyz=0.025 -0.043 0 rpy=0 0 0

Commit message: Enable deformable finger contact with CB/FEM objects and double finger length.
Wire contact_deformable_gripper to all grasp targets, add finger↔deformable-box penalty contact, shift the grasp box for 160 mm prongs, and align object Young's modulus at 3e4 Pa.

Co-authored-by: Cursor <cursoragent@cursor.com>

File: examples/pure_simulation/urdf/arm6_gripper/arm6_gripper.urdf (robot description, URDF)
Before this commit: robot arm6_gripper, 8 links, 7 joints
Links:
- link left_finger: mass 0.12 -> 0.24; geometry collision box size=0.160 0.010 0.040; visual box size=0.160 0.010 0.040
- link right_finger: mass 0.12 -> 0.24; geometry collision box size=0.160 0.010 0.040; visual box size=0.160 0.010 0.040
